File: alim_board/alim_board.kicad_pcb (KiCad board)
At the start: 2 copper layers, 37 x 40 mm, 14 parts, among them J1 Alimentation, J2 Conn_01x02, J3 Conn_01x02, J4 Conn_01x02, J5 Conn_01x02, J6 Conn_01x02

Commit message: Improve pads-zones connections and silkscreen. Add a step file of the pcb
Parts:
- added G***: LOGO, Logos:pollen_xsmall, F.Cu at (124.8, 64.5)
Routing:
- net GND: track 0.00 -> 22.2 mm
- net VCC: track 0.00 -> 12.6 mm
- net Net-(H4-Pad1): track 0.00 -> 12.3 mm
- net Net-(H3-Pad1): track 0.00 -> 5.70 mm
Other:
- board text added: "+12V"
- board text added: "alim-board 1.0.1"
- board text removed: "Vcc +12V"
